Commit message: up

File: celconv_description/urdf/celconv_rim.urdf.xacro (robot description, xacro)
@@ -85,4 +85,14 @@
   	  rpy="-1.570796326794896 0 -0.7853981633974483"
   	/>
+	<transmission name="rim_${name}_${parent_name}_transmission">
+	  <type>transmission_interface/SimpleTransmission</type>
+	  <joint name="rim_${name}_to_${parent_name}_joint">
+	    <hardwareInterface>hardware_interface/VelocityJointInterface</hardwareInterface>
+	  </joint>
+	  <actuator name="rim_${name}_${parent_name}_motor">
+	    <hardwareInterface>hardware_interface/VelocityJointInterface</hardwareInterface>
+	    <mechanicalReduction>1</mechanicalReduction>
+	  </actuator>
+	</transmission>
   </xacro:macro>
 </robot>

File: celconv_description/urdf/celconv_roller.urdf.xacro (robot description, xacro)
@@ -22,4 +22,12 @@
   	</visual>
   	<collision>
+	  <!-- <surface>
+	    <friction>
+	      <ode>
+	        <mu>0.5</mu>
+	        <mu2>0.5</mu2>
+	      </ode>
+	    </friction>
+	  </surface> -->
   	  <geometry>
   	  	<mesh filename="file://$(find celconv_description)/mesh/celconv_roller.stl"/>
