Commit message: commit

File: celconv_description/urdf/celconv_cell.urdf.xacro (robot description, xacro)
@@ -2,6 +2,6 @@
 <robot xmlns:xacro="http://www.ros.org/wiki/xacro">
   <xacro:include filename="$(find celconv_description)/urdf/celconv_rim.urdf.xacro"/>
-  <xacro:macro name="celconv_cell" params="name">
-    <link name="${name}_link">
+  <xacro:macro name="celconv_cell" params="name parent_name color xyz rpy">
+    <link name="cell_${name}_${parent_name}_link">
       <inertial>
         <mass value="0.07862944645"/>
@@ -18,6 +18,6 @@
           <mesh filename="file://$(find celconv_description)/mesh/celconv_base.stl"/>
         </geometry>
-        <material name="base_material">
-          <color rgba="1 1 1 1"/>
+        <material name="cell_${name}_${parent_name}_material">
+          <color rgba="${color} 1"/>
         </material>
       </visual>
@@ -28,9 +28,30 @@
       </collision>
     </link>
+    <joint
+  	  name="cell_${name}_to_${parent_name}_joint"
+  	  type="fixed">
+  	  <parent link="${parent_name}_link" />
+  	  <child link="cell_${name}_${parent_name}_link" />
+  	  <axis xyz="0 0 0"/>
+  	  <origin xyz="${xyz}" rpy="${rpy}"/>
+  	</joint>
     <xacro:celconv_rim
 		  name="left"
+      parent_name="cell_${name}_${parent_name}"
 		  color="0.3 0 0"
-		  xyz="-0.03464101615 0.02 0.2"
+		  xyz="-0.0671 0.03875 0.095"
 		  rpy="1.570796326794896 0 1.047197551196597"/>
+	  <xacro:celconv_rim
+	  	name="back"
+      parent_name="cell_${name}_${parent_name}"
+	  	color="0 0.3 0"
+	  	xyz="0 -0.0775 0.095"
+	  	rpy="1.570796326794896 0 3.141592653589793"/>
+	  <xacro:celconv_rim
+	  	name="right"
+      parent_name="cell_${name}_${parent_name}"
+	  	color="0 0 0.3"
+	  	xyz="0.0671 0.03875 0.095"
+	  	rpy="1.570796326794896 0 -1.047197551196597"/>
   </xacro:macro>
 </robot>

File: celconv_description/urdf/celconv_main.urdf.xacro (robot description, xacro)
@@ -10,4 +10,5 @@
   <xacro:property name="row" value="0"/>
   <xacro:property name="col" value="0"/>
+  <link name="base_link"></link>
   <!-- Define a macro to handle cell creation and joint connection -->
   <xacro:macro name="create_cells" params="row col num_rows num_cols">
@@ -23,11 +24,9 @@
       <xacro:if value="${col &lt; num_cols}">
         <xacro:property name="cell_index" value="${row * num_cols + col}"/>
-        <xacro:celconv_cell name="cell_${cell_index}"/>
-        <joint name="joint_${cell_index}" type="fixed">
-          <parent link="base_link"/>
-          <child link="cell_${cell_index}_link"/>
-          <!-- Adjust origin based on row parity and column position -->
-          <origin xyz="${col * col_dist + (row % 2) * (col_dist / 2)} ${y} 0"/>
-        </joint>
+        <xacro:celconv_cell name="${cell_index}"
+                            parent_name="base"
+                            color="1 1 1"
+                            xyz="${col * col_dist + (row % 2) * (col_dist / 2)} ${y} 0"
+                            rpy="0 0 0"/>
         <!-- Recurse for the next column -->
         <xacro:create_cells row="${row}" col="${col + 1}" num_rows="${num_rows}" num_cols="${num_cols}"/>
@@ -41,9 +40,3 @@
   <!-- Start the cell creation process -->
   <xacro:create_cells row="${row}" col="${col}" num_rows="${num_rows}" num_cols="${num_cols}"/>
-  <link name="base_link"></link>
-  <joint name="base_to_cell_0_joint" type="fixed">
-    <parent link="base_link"/>
-    <child link="cell_0_link"/>
-    <origin xyz="0 0 0"/>
-  </joint>
 </robot>

File: celconv_description/urdf/celconv_rim.urdf.xacro (robot description, xacro)
@@ -1,6 +1,7 @@
 <?xml version="1.0" ?>
 <robot xmlns:xacro="http://www.ros.org/wiki/xacro">
-  <xacro:macro name="celconv_rim"  params="name color xyz rpy">
-  	<link name="rim_${name}_link">
+  <xacro:include filename="$(find celconv_description)/urdf/celconv_roller.urdf.xacro"/>
+  <xacro:macro name="celconv_rim"  params="name parent_name color xyz rpy">
+  	<link name="rim_${name}_${parent_name}_link">
   	  <inertial>
   	  	<origin xyz="0 0 -0.000343"/>
@@ -18,5 +19,5 @@
   	  		<mesh filename="file://$(find celconv_description)/mesh/celconv_rim.stl"/>
   	  	</geometry>
-  	  	<material name="rim_${name}_material">
+  	  	<material name="rim_${name}_${parent_name}_material">
   	  		<color rgba="${color} 1"/>
   	  	</material>
@@ -29,11 +30,59 @@
   	</link>
   	<joint
-  	  name="rim_${name}_joint"
+  	  name="rim_${name}_to_${parent_name}_joint"
   	  type="continuous">
-  	  <parent link="${name}_link" />
-  	  <child link="rim_${name}_link" />
+  	  <parent link="${parent_name}_link" />
+  	  <child link="rim_${name}_${parent_name}_link" />
   	  <axis xyz="0 0 1"/>
   	  <origin xyz="${xyz}" rpy="${rpy}"/>
   	</joint>
+  	<xacro:celconv_roller
+  	  parent_name="rim_${name}_${parent_name}"
+  	  name="e"
+  	  xyz="0.01355 0 0.0055"
+  	  rpy="-1.570796326794896 0 0"
+  	/>
+  	<xacro:celconv_roller
+  	  parent_name="rim_${name}_${parent_name}"
+  	  name="ne"
+  	  xyz="0.00958129689 0.00958129689 -0.0055"
+  	  rpy="-1.570796326794896 0 0.7853981633974483"
+  	/>
+  	<xacro:celconv_roller
+  	  parent_name="rim_${name}_${parent_name}"
+  	  name="n"
+  	  xyz="0 0.01355 0.0055"
+  	  rpy="-1.570796326794896 0 1.570796326794896"
+  	/>
+  	<xacro:celconv_roller
+  	  parent_name="rim_${name}_${parent_name}"
+  	  name="nw"
+  	  xyz="-0.00958129689 0.00958129689 -0.0055"
+  	  rpy="-1.570796326794896 0 2.356194490192345"
+  	/>
+  	<xacro:celconv_roller
+  	  parent_name="rim_${name}_${parent_name}"
+  	  name="w"
+  	  xyz="-0.01355 0 0.0055"
+  	  rpy="-1.570796326794896 0 3.141592653589793"
+  	/>
+  	<xacro:celconv_roller
+  	  parent_name="rim_${name}_${parent_name}"
+  	  name="sw"
+  	  xyz="-0.00958129689 -0.00958129689 -0.0055"
+  	  rpy="-1.570796326794896 0 -2.356194490192345"
+  	/>
+  	<xacro:celconv_roller
+  	  parent_name="rim_${name}_${parent_name}"
+  	  name="s"
+  	  xyz="0 -0.01355 0.0055"
+  	  rpy="-1.570796326794896 0 -1.570796326794896"
+  	/>
+  	<xacro:celconv_roller
+  	  parent_name="rim_${name}_${parent_name}"
+  	  name="se"
+  	  xyz="0.00958129689 -0.00958129689 -0.0055"
+  	  rpy="-1.570796326794896 0 -0.7853981633974483"
+  	/>
   </xacro:macro>
 </robot>

Commit message: up

File: celconv_description/urdf/celconv_cell.urdf.xacro (robot description, xacro)
@@ -54,4 +54,24 @@
 	  	xyz="0.0671 0.03875 0.095"
 	  	rpy="1.570796326794896 0 -1.047197551196597"/>
+  	<!-- <ros2_control name="cell_${name}_${parent_name}_GazeboSystem" type="system">
+  	  <hardware>
+  	    <plugin>gazebo_ros2_control/GazeboSystem</plugin>
+  	  </hardware>
+	    <joint name="rim_left_to_${name}_${parent_name}_joint">
+        	<command_interface name="velocity"/>
+        	<state_interface name="position"/>
+        	<state_interface name="velocity"/>
+	    </joint>
+	    <joint name="rim_back_to_${name}_${parent_name}_joint">
+        	<command_interface name="velocity"/>
+        	<state_interface name="position"/>
+        	<state_interface name="velocity"/>
+	    </joint>
+	    <joint name="rim_right_to_${name}_${parent_name}_joint">
+        	<command_interface name="velocity"/>
+        	<state_interface name="position"/>
+        	<state_interface name="velocity"/>
+	    </joint>
+  	</ros2_control> -->
   </xacro:macro>
 </robot>

File: celconv_description/urdf/celconv_main.urdf.xacro (robot description, xacro)
@@ -3,9 +3,11 @@
   <xacro:include filename="$(find celconv_description)/urdf/celconv_cell.urdf.xacro"/>
   <!-- Define the number of rows and columns as input -->
+  <!-- <xacro:arg name="num_rows" default="2"/>
+  <xacro:arg name="num_cols" default="2"/> -->
   <xacro:property name="num_rows" value="$(arg num_rows)"/>
   <xacro:property name="num_cols" value="$(arg num_cols)"/>
   <xacro:property name="dist_bias" value="0.005"/>
-  <xacro:property name="row_dist" value="${dist_bias + 0.1}"/>
-  <xacro:property name="col_dist" value="${dist_bias + 0.11547 * 3}"/>
+  <xacro:property name="row_dist" value="${dist_bias + 0.2}"/>
+  <xacro:property name="col_dist" value="${dist_bias + 0.11547 * 1.5}"/>
   <xacro:property name="row" value="0"/>
   <xacro:property name="col" value="0"/>
@@ -20,5 +22,5 @@
     <xacro:if value="${row &lt; num_rows}">
       <!-- Calculate y position -->
-      <xacro:property name="y" value="${row * row_dist}"/>
+      <xacro:property name="y" value="${row * row_dist + (col % 2) * (row_dist / 2)}"/>
       <!-- Handle cells in the current row -->
       <xacro:if value="${col &lt; num_cols}">
@@ -27,5 +29,5 @@
                             parent_name="base"
                             color="1 1 1"
-                            xyz="${col * col_dist + (row % 2) * (col_dist / 2)} ${y} 0"
+                            xyz="${col * col_dist} ${y} 0"
                             rpy="0 0 0"/>
         <!-- Recurse for the next column -->
@@ -40,3 +42,28 @@
   <!-- Start the cell creation process -->
   <xacro:create_cells row="${row}" col="${col}" num_rows="${num_rows}" num_cols="${num_cols}"/>
+  <!-- <ros2_control name="cell_0_base_GazeboSystem" type="system">
+    <hardware>
+      <plugin>gazebo_ros2_control/GazeboSystem</plugin>
+    </hardware>
+	  <joint name="rim_left_to_0_base_joint">
+      	<command_interface name="velocity"/>
+      	<state_interface name="position"/>
+      	<state_interface name="velocity"/>
+	  </joint>
+	  <joint name="rim_back_to_0_base_joint">
+      	<command_interface name="velocity"/>
+      	<state_interface name="position"/>
+      	<state_interface name="velocity"/>
+	  </joint>
+	  <joint name="rim_right_to_0_base_joint">
+      	<command_interface name="velocity"/>
+      	<state_interface name="position"/>
+      	<state_interface name="velocity"/>
+	  </joint>
+  </ros2_control>
+  <gazebo>
+    <plugin filename="libgazebo_ros2_control.so" name="gazebo_ros2_control">
+      <parameters>$(find celconv_control)/config/celconv_gazebo_controller_velocity.yaml</parameters>
+    </plugin>
+  </gazebo> -->
 </robot>

Commit message: up

File: celconv_description/urdf/celconv_cell.urdf.xacro (robot description, xacro)
@@ -54,24 +54,24 @@
 	  	xyz="0.0671 0.03875 0.095"
 	  	rpy="1.570796326794896 0 -1.047197551196597"/>
-  	<!-- <ros2_control name="cell_${name}_${parent_name}_GazeboSystem" type="system">
+  	<ros2_control name="cell_${name}_${parent_name}_hardware" type="system">
   	  <hardware>
   	    <plugin>gazebo_ros2_control/GazeboSystem</plugin>
   	  </hardware>
-	    <joint name="rim_left_to_${name}_${parent_name}_joint">
+	    <joint name="rim_left_to_cell_${name}_${parent_name}_joint">
         	<command_interface name="velocity"/>
         	<state_interface name="position"/>
         	<state_interface name="velocity"/>
 	    </joint>
-	    <joint name="rim_back_to_${name}_${parent_name}_joint">
+	    <joint name="rim_back_to_cell_${name}_${parent_name}_joint">
         	<command_interface name="velocity"/>
         	<state_interface name="position"/>
         	<state_interface name="velocity"/>
 	    </joint>
-	    <joint name="rim_right_to_${name}_${parent_name}_joint">
+	    <joint name="rim_right_to_cell_${name}_${parent_name}_joint">
         	<command_interface name="velocity"/>
         	<state_interface name="position"/>
         	<state_interface name="velocity"/>
 	    </joint>
-  	</ros2_control> -->
+  	</ros2_control>
   </xacro:macro>
 </robot>

File: celconv_description/urdf/celconv_main.urdf.xacro (robot description, xacro)
@@ -5,4 +5,5 @@
   <!-- <xacro:arg name="num_rows" default="2"/>
   <xacro:arg name="num_cols" default="2"/> -->
+  <xacro:arg name="control_cfg_prefix" default="celconv"/>
   <xacro:property name="num_rows" value="$(arg num_rows)"/>
   <xacro:property name="num_cols" value="$(arg num_cols)"/>
@@ -22,5 +23,7 @@
     <xacro:if value="${row &lt; num_rows}">
       <!-- Calculate y position -->
-      <xacro:property name="y" value="${row * row_dist + (col % 2) * (row_dist / 2)}"/>
+      <xacro:property name="y" value="${row * row_dist - (col % 2) * (row_dist / 2)}"/>
+      <xacro:property name="x" value="${col * col_dist}"/>
+      <xacro:property name="z" value="0"/>
       <!-- Handle cells in the current row -->
       <xacro:if value="${col &lt; num_cols}">
@@ -29,5 +32,5 @@
                             parent_name="base"
                             color="1 1 1"
-                            xyz="${col * col_dist} ${y} 0"
+                            xyz="${x} ${y} ${z}"
                             rpy="0 0 0"/>
         <!-- Recurse for the next column -->
@@ -42,28 +45,8 @@
   <!-- Start the cell creation process -->
   <xacro:create_cells row="${row}" col="${col}" num_rows="${num_rows}" num_cols="${num_cols}"/>
-  <!-- <ros2_control name="cell_0_base_GazeboSystem" type="system">
-    <hardware>
-      <plugin>gazebo_ros2_control/GazeboSystem</plugin>
-    </hardware>
-	  <joint name="rim_left_to_0_base_joint">
-      	<command_interface name="velocity"/>
-      	<state_interface name="position"/>
-      	<state_interface name="velocity"/>
-	  </joint>
-	  <joint name="rim_back_to_0_base_joint">
-      	<command_interface name="velocity"/>
-      	<state_interface name="position"/>
-      	<state_interface name="velocity"/>
-	  </joint>
-	  <joint name="rim_right_to_0_base_joint">
-      	<command_interface name="velocity"/>
-      	<state_interface name="position"/>
-      	<state_interface name="velocity"/>
-	  </joint>
-  </ros2_control>
   <gazebo>
     <plugin filename="libgazebo_ros2_control.so" name="gazebo_ros2_control">
-      <parameters>$(find celconv_control)/config/celconv_gazebo_controller_velocity.yaml</parameters>
+      <parameters>$(find celconv_control)/config/$(arg control_cfg_prefix)_gazebo_control.yaml</parameters>
     </plugin>
-  </gazebo> -->
+  </gazebo>
 </robot>

Commit message: up

File: celconv_description/urdf/celconv_cell.urdf.xacro (robot description, xacro)
@@ -2,8 +2,8 @@
 <robot xmlns:xacro="http://www.ros.org/wiki/xacro">
   <xacro:include filename="$(find celconv_description)/urdf/celconv_rim.urdf.xacro"/>
-  <xacro:macro name="celconv_cell" params="name parent_name color xyz rpy">
+  <xacro:macro name="celconv_cell" params="name parent_name color xyz rpy is_sim">
     <link name="cell_${name}_${parent_name}_link">
       <inertial>
-        <mass value="0.07862944645"/>
+        <mass value="1"/>
         <inertia
           ixx="0"
@@ -56,5 +56,7 @@
   	<ros2_control name="cell_${name}_${parent_name}_hardware" type="system">
   	  <hardware>
-  	    <plugin>gazebo_ros2_control/GazeboSystem</plugin>
+	  	<xacro:if value="${is_sim}">
+  	    	<plugin>gazebo_ros2_control/GazeboSystem</plugin>
+		</xacro:if>
   	  </hardware>
 	    <joint name="rim_left_to_cell_${name}_${parent_name}_joint">

File: celconv_description/urdf/celconv_main.urdf.xacro (robot description, xacro)
@@ -3,9 +3,12 @@
   <xacro:include filename="$(find celconv_description)/urdf/celconv_cell.urdf.xacro"/>
   <!-- Define the number of rows and columns as input -->
-  <!-- <xacro:arg name="num_rows" default="2"/>
-  <xacro:arg name="num_cols" default="2"/> -->
-  <xacro:arg name="control_cfg_prefix" default="celconv"/>
+  <xacro:arg name="num_rows" default="2"/>
+  <xacro:arg name="num_cols" default="2"/>
+  <xacro:arg name="is_sim" default="false"/>
+  <xacro:arg name="prefix" default=""/>
+  <xacro:property name="is_sim" value="$(arg is_sim)"/>
   <xacro:property name="num_rows" value="$(arg num_rows)"/>
   <xacro:property name="num_cols" value="$(arg num_cols)"/>
+  <!-- Define the distance between cells -->
   <xacro:property name="dist_bias" value="0.005"/>
   <xacro:property name="row_dist" value="${dist_bias + 0.2}"/>
@@ -33,5 +36,6 @@
                             color="1 1 1"
                             xyz="${x} ${y} ${z}"
-                            rpy="0 0 0"/>
+                            rpy="0 0 0"
+                            is_sim="$(arg is_sim)"/>
         <!-- Recurse for the next column -->
         <xacro:create_cells row="${row}" col="${col + 1}" num_rows="${num_rows}" num_cols="${num_cols}"/>
@@ -45,8 +49,10 @@
   <!-- Start the cell creation process -->
   <xacro:create_cells row="${row}" col="${col}" num_rows="${num_rows}" num_cols="${num_cols}"/>
-  <gazebo>
-    <plugin filename="libgazebo_ros2_control.so" name="gazebo_ros2_control">
-      <parameters>$(find celconv_control)/config/$(arg control_cfg_prefix)_gazebo_control.yaml</parameters>
-    </plugin>
-  </gazebo>
+  <xacro:if value="$(arg is_sim)">
+    <gazebo>
+      <plugin filename="libgazebo_ros2_control.so" name="gazebo_ros2_control">
+        <parameters>$(find celconv_control)/config/$(arg prefix)_gazebo_control.yaml</parameters>
+      </plugin>
+    </gazebo>
+  </xacro:if>
 </robot>

Commit message: up

File: celconv_description/urdf/celconv_cell.urdf.xacro (robot description, xacro)
@@ -5,5 +5,5 @@
     <link name="cell_${name}_${parent_name}_link">
       <inertial>
-        <mass value="1"/>
+        <mass value="2.0"/>
         <inertia
           ixx="0"

File: celconv_description/urdf/celconv_roller.urdf.xacro (robot description, xacro)
@@ -22,12 +22,12 @@
   	</visual>
   	<collision>
-	  <!-- <surface>
+	  <surface>
 	    <friction>
 	      <ode>
-	        <mu>0.5</mu>
-	        <mu2>0.5</mu2>
+	        <mu>1.0</mu>
+	        <mu2>1.0</mu2>
 	      </ode>
 	    </friction>
-	  </surface> -->
+	  </surface>
   	  <geometry>
   	  	<mesh filename="file://$(find celconv_description)/mesh/celconv_roller.stl"/>

File: celconv_gazebo/urdf/box.urdf.xacro (robot description, xacro)
@@ -2,7 +2,7 @@
 <robot xmlns:xacro="http://ros.org/wiki/xacro" name="small_box">
   <!-- Define the dimensions as Xacro properties -->
-  <xacro:property name="height" value="0.23094"/>
-  <xacro:property name="width" value="0.23094"/>
-  <xacro:property name="depth" value="0.11547"/> <!-- Assuming depth is the same as width for simplicity -->
+  <xacro:property name="height" value="0.3"/>
+  <xacro:property name="width" value="0.3"/>
+  <xacro:property name="depth" value="0.1"/> <!-- Assuming depth is the same as width for simplicity -->
   <!-- Link for the box -->
   <link name="box_link">
@@ -16,7 +16,15 @@
         <box size="${width} ${height} ${depth}"/>
       </geometry>
+      <surface>
+        <friction>
+          <ode>
+            <mu>0.3</mu>  <!-- Typical friction coefficient for cardboard -->
+            <mu2>0.3</mu2>
+          </ode>
+        </friction>
+      </surface>
     </collision>
     <inertial>
-      <mass value="0.05"/> <!-- Assuming some mass for the box -->
+      <mass value="0.0005"/> <!-- Assuming some mass for the box -->
       <inertia ixx="0.1" ixy="0" ixz="0" iyy="0.1" iyz="0" izz="0.1"/>
     </inertial>

Commit message: up

File: celconv_description/urdf/celconv_cell.urdf.xacro (robot description, xacro)
@@ -40,5 +40,5 @@
       parent_name="cell_${name}_${parent_name}"
 		  color="0.3 0 0"
-		  xyz="-0.0671 0.03875 0.095"
+		  xyz="-0.03507 0.02025 0.095"
 		  rpy="1.570796326794896 0 1.047197551196597"/>
 	  <xacro:celconv_rim
@@ -46,5 +46,5 @@
       parent_name="cell_${name}_${parent_name}"
 	  	color="0 0.3 0"
-	  	xyz="0 -0.0775 0.095"
+	  	xyz="0 -0.0405 0.095"
 	  	rpy="1.570796326794896 0 3.141592653589793"/>
 	  <xacro:celconv_rim
@@ -52,5 +52,5 @@
       parent_name="cell_${name}_${parent_name}"
 	  	color="0 0 0.3"
-	  	xyz="0.0671 0.03875 0.095"
+	  	xyz="0.03507 0.02025 0.095"
 	  	rpy="1.570796326794896 0 -1.047197551196597"/>
   	<ros2_control name="cell_${name}_${parent_name}_hardware" type="system">

File: celconv_description/urdf/celconv_main.urdf.xacro (robot description, xacro)
@@ -11,7 +11,7 @@
   <xacro:property name="num_cols" value="$(arg num_cols)"/>
   <!-- Define the distance between cells -->
-  <xacro:property name="dist_bias" value="0.005"/>
-  <xacro:property name="row_dist" value="${dist_bias + 0.2}"/>
-  <xacro:property name="col_dist" value="${dist_bias + 0.11547 * 1.5}"/>
+  <xacro:property name="dist_bias" value="0.000"/>
+  <xacro:property name="row_dist" value="${dist_bias + 0.12}"/>
+  <xacro:property name="col_dist" value="${dist_bias + 0.06928 * 1.5}"/>
   <xacro:property name="row" value="0"/>
   <xacro:property name="col" value="0"/>
